Commit message: fix(model): recalibrate wheel separation and update collision geometry

File: src/JetRover/jetrover_description/urdf/car_mecanum.urdf.xacro (robot description, xacro)
@@ -62,10 +62,7 @@
     </visual>
     <collision>
-      <origin
-        xyz="0 0 0"
-        rpy="0 0 0" />
-      <geometry>
-        <mesh
-          filename="package://jetrover_description/meshes/mecanum/wheel_left_front_link_collision.stl" />
+      <origin xyz="0 0 0" rpy="${M_PI/2} 0 0" />
+      <geometry>
+        <cylinder radius="0.04825" length="0.035"/>
       </geometry>
     </collision>
@@ -111,10 +108,7 @@
     </visual>
     <collision>
-      <origin
-        xyz="0 0 0"
-        rpy="0 0 0" />
-      <geometry>
-        <mesh
-          filename="package://jetrover_description/meshes/mecanum/wheel_left_back_link_collision.stl" />
+      <origin xyz="0 0 0" rpy="${M_PI/2} 0 0" />
+      <geometry>
+        <cylinder radius="0.04825" length="0.035"/>
       </geometry>
     </collision>
@@ -160,10 +154,7 @@
     </visual>
     <collision>
-      <origin
-        xyz="0 0 0"
-        rpy="0 0 0" />
-      <geometry>
-        <mesh
-            filename="package://jetrover_description/meshes/mecanum/wheel_right_front_link_collision.stl" />
+      <origin xyz="0 0 0" rpy="${M_PI/2} 0 0" />
+      <geometry>
+        <cylinder radius="0.04825" length="0.035"/>
       </geometry>
     </collision>
@@ -209,10 +200,7 @@
     </visual>
     <collision>
-      <origin
-        xyz="0 0 0"
-        rpy="0 0 0" />
-      <geometry>
-        <mesh
-            filename="package://jetrover_description/meshes/mecanum/wheel_right_back_link_collision.stl" />
+      <origin xyz="0 0 0" rpy="${M_PI/2} 0 0" />
+      <geometry>
+        <cylinder radius="0.04825" length="0.035"/>
       </geometry>
     </collision>

File: src/JetRover/jetrover_description/urdf/jetrover_gazebo.xacro (robot description, xacro)
@@ -2,5 +2,5 @@
 <robot xmlns:xacro="http://ros.org/wiki/xacro">
   <!-- 1. 底盤全向移動外掛 (Mecanum Drive) -->
-  <gazebo>
+   <gazebo>
     <plugin
       filename="gz-sim-mecanum-drive-system"
@@ -10,17 +10,52 @@
       <front_right_joint>wheel_right_front_joint</front_right_joint>
       <back_right_joint>wheel_right_back_joint</back_right_joint>
-      <wheel_separation>0.22426</wheel_separation>
+      <wheel_separation>0.1412</wheel_separation>
       <wheel_base>0.19503</wheel_base>
       <wheel_radius>0.048</wheel_radius>
       <topic>/cmd_vel</topic>
-      <odom_topic>/odom</odom_topic>
-      <tf_topic>/tf</tf_topic>
+      <!-- 修改 topic 避免與真實位姿 odom 衝突 -->
+      <odom_topic>/wheel_odom</odom_topic>
+      <tf_topic>/wheel_tf</tf_topic>
       <frame_id>odom</frame_id>
       <child_frame_id>base_footprint</child_frame_id>
     </plugin>
   </gazebo>
+  <!-- 2. 物理真值里程計外掛 (直接讀取 Gazebo 世界位姿，撞牆會即時停止) -->
+  <gazebo>
+    <plugin
+      filename="gz-sim-odometry-publisher-system"
+      name="gz::sim::systems::OdometryPublisher">
+      <odom_frame>odom</odom_frame>
+      <robot_base_frame>base_footprint</robot_base_frame>
+      <odom_topic>/odom</odom_topic>
+      <tf_topic>/tf</tf_topic>
+      <dimensions>2</dimensions>
+      <odom_publish_frequency>50</odom_publish_frequency>
+    </plugin>
+  </gazebo>
+  <!-- 請針對 4 個輪子 (wheel_left_front_link, wheel_left_back_link, wheel_right_front_link, wheel_right_back_link) 分別加入： -->
   <gazebo reference="wheel_left_front_link">
-    <mu1>0.2</mu1>
-    <mu2>0.2</mu2>
+    <mu1>0.1</mu1>
+    <mu2>0.1</mu2>
+    <kp>1000000.0</kp>
+    <kd>1.0</kd>
+  </gazebo>
+  <gazebo reference="wheel_left_back_link">
+    <mu1>0.1</mu1>
+    <mu2>0.1</mu2>
+    <kp>1000000.0</kp>
+    <kd>1.0</kd>
+  </gazebo>
+  <gazebo reference="wheel_right_front_link">
+    <mu1>0.1</mu1>
+    <mu2>0.1</mu2>
+    <kp>1000000.0</kp>
+    <kd>1.0</kd>
+  </gazebo>
+  <gazebo reference="wheel_right_back_link">
+    <mu1>0.1</mu1>
+    <mu2>0.1</mu2>
+    <kp>1000000.0</kp>
+    <kd>1.0</kd>
   </gazebo>
   <!-- 2. 輪子關節狀態廣播外掛 (Joint State Publisher) -->
